Commit message: fix(urdf): align LiDAR forward mathematically to fix odometry scan-matching mismatch

File: titan_ws/src/titan_description/urdf/lidar.xacro (robot description, xacro)
@@ -4,5 +4,5 @@
         <parent link="chassis"/>
         <child link="laser_frame"/>
-        <origin xyz="0.2 0 0.1" rpy="0 0 3.14159"/>
+        <origin xyz="0.2 0 0.1" rpy="0 0 0"/>
     </joint>
     <link name="laser_frame">

Commit message: fix(physics): resolve motor low-voltage stall by increasing default velocity and revert URDF/Odometry polarities

File: titan_ws/src/titan_description/urdf/lidar.xacro (robot description, xacro)
@@ -4,5 +4,5 @@
         <parent link="chassis"/>
         <child link="laser_frame"/>
-        <origin xyz="0.2 0 0.1" rpy="0 0 0"/>
+        <origin xyz="0.2 0 0.1" rpy="0 0 3.14159"/>
     </joint>
     <link name="laser_frame">
